File: PCB/Adafruit-HUZZAH32-ESP32-Feather-PCB-master/Adafruit HUZZAH32 ESP32 Feather.brd (EAGLE design)
At the start: 50.8 x 22.9 mm, 41 parts, among them IC1 CP2104, Q1 mmbt2222, Q2 mmbt2222, Q3 DMG3415U, SW2 KMR2, U2 AP2112-3.3, U3 MCP73831T-2ACI/OT, X1 JSTPH, X2 ESP32_WROOM32_SKINNY, X4 20329

Commit message: dsasd
Parts:
- removed DIS1: TUXGR_16X2_R2, display-lcd:TUXGR_16X2_R2
Connections:
- removed net VCC: DIS1.2
- net GND: no longer DIS1.1
Changed lines of the file:
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@@
 <grid distance="0.0025" unitdist="inch" unit="inch" style="lines" multiple="1" display="no" altdistance="0.025" altunitdist="inch" altunit="inch"/>
 <layers>
-<layer number="1" name="Top" color="4" fill="1" visible="yes" active="yes"/>
+<layer number="1" name="Top" color="4" fill="1" visible="no" active="yes"/>
 <layer number="2" name="Route2" color="1" fill="3" visible="no" active="no"/>
 <layer number="3" name="Route3" color="4" fill="3" visible="no" active="no"/>
@@
 <layer number="14" name="Route14" color="1" fill="6" visible="no" active="no"/>
 <layer number="15" name="Route15" color="4" fill="6" visible="no" active="no"/>
-<layer number="16" name="Bottom" color="1" fill="1" visible="yes" active="yes"/>
+<layer number="16" name="Bottom" color="1" fill="1" visible="no" active="yes"/>
 <layer number="17" name="Pads" color="2" fill="1" visible="yes" active="yes"/>
-<layer number="18" name="Vias" color="2" fill="1" visible="yes" active="yes"/>
-<layer number="19" name="Unrouted" color="6" fill="1" visible="yes" active="yes"/>
-<layer number="20" name="Dimension" color="15" fill="1" visible="yes" active="yes"/>
-<layer number="21" name="tPlace" color="14" fill="1" visible="yes" active="yes"/>
+<layer number="18" name="Vias" color="2" fill="1" visible="no" active="yes"/>
+<layer number="19" name="Unrouted" color="6" fill="1" visible="no" active="yes"/>
+<layer number="20" name="Dimension" color="15" fill="1" visible="no" active="yes"/>
+<layer number="21" name="tPlace" color="14" fill="1" visible="no" active="yes"/>
 <layer number="22" name="bPlace" color="13" fill="1" visible="no" active="yes"/>
-<layer number="23" name="tOrigins" color="14" fill="1" visible="yes" active="yes"/>
+<layer number="23" name="tOrigins" color="14" fill="1" visible="no" active="yes"/>
 <layer number="24" name="bOrigins" color="13" fill="1" visible="no" active="yes"/>
 <layer number="25" name="tNames" color="7" fill="1" visible="no" active="yes"/>
@@
 <layer number="43" name="vRestrict" color="2" fill="10" visible="no" active="yes"/>
 <layer number="44" name="Drills" color="7" fill="1" visible="no" active="yes"/>
-<layer number="45" name="Holes" color="7" fill="1" visible="yes" active="yes"/>
+<layer number="45" name="Holes" color="7" fill="1" visible="no" active="yes"/>
 <layer number="46" name="Milling" color="3" fill="1" visible="no" active="yes"/>
-<layer number="47" name="Measures" color="7" fill="1" visible="yes" active="yes"/>
+<layer number="47" name="Measures" color="7" fill="1" visible="no" active="yes"/>
 <layer number="48" name="Document" color="7" fill="1" visible="no" active="yes"/>
 <layer number="49" name="Reference" color="7" fill="1" visible="no" active="yes"/>
@@
 <element name="U$9" library="silks" package="FEATHERLOGO_MED" value="" x="24.13" y="7.493" smashed="yes" rot="MR0"/>
 <element name="U$43" library="silks" package="HUZZAH32" value="" x="50.3555" y="10.8585" smashed="yes" rot="MR0"/>
-<element name="DIS1" library="display-lcd" library_urn="urn:adsk.eagle:library:214" package="TUXGR_16X2_R2" package3d_urn="urn:adsk.eagle:package:13139/1" value="TUXGR_16X2_R2" x="0" y="0" smashed="yes">
-<attribute name="MF" value="" x="0" y="0" size="1.778" layer="27" display="off"/>
-<attribute name="MPN" value="" x="0" y="0" size="1.778" layer="27" display="off"/>
-<attribute name="NAME" x="-38.1" y="18.415" size="1.27" layer="25"/>
-<attribute name="OC_FARNELL" value="unknown" x="0" y="0" size="1.778" layer="27" display="off"/>
-<attribute name="OC_NEWARK" value="unknown" x="0" y="0" size="1.778" layer="27" display="off"/>
-<attribute name="POPULARITY" value="5" x="0" y="0" size="1.778" layer="27" display="off"/>
-<attribute name="VALUE" x="0.635" y="18.415" size="1.27" layer="27"/>
-</element>
 </elements>
 <signals>
@@
 <via x="33.4645" y="18.0975" extent="1-16" drill="0.5"/>
 <via x="31.1785" y="22.7965" extent="1-16" drill="0.5"/>
-<contactref element="DIS1" pad="1"/>
 <wire x1="48.0695" y1="30.1625" x2="47.6085" y2="31.6775" width="0" layer="19" extent="1-1"/>
 <wire x1="48.1965" y1="27.6225" x2="48.0695" y2="30.1625" width="0" layer="19" extent="1-1"/>
@@
 <wire x1="25.0825" y1="17.8435" x2="21.5265" y2="18.2245" width="0" layer="19" extent="1-1"/>
 <wire x1="9.0805" y1="12.6365" x2="10.3505" y2="17.4625" width="0" layer="19" extent="1-1"/>
-<wire x1="-32" y1="15.5" x2="6.7995" y2="19.5775" width="0" layer="19" extent="1-1"/>
 </signal>
 <signal name="VBUS">
@@
 <wire x1="43.6245" y1="33.1851" x2="43.6245" y2="33.3375" width="0.254" layer="16"/>
 </signal>
-<signal name="VCC">
-<contactref element="DIS1" pad="2"/>
-</signal>
 </signals>
 <mfgpreviewcolors>
@@
 which will not be processed correctly with this version.
 </note>
-<note version="8.2" severity="warning">
-Since Version 8.2, EAGLE supports online libraries. The ids
-of those online libraries will not be understood (or retained)
-with this version.
-</note>
-<note version="8.3" severity="warning">
-Since Version 8.3, EAGLE supports URNs for individual library
-assets (packages, symbols, and devices). The URNs of those assets
-will not be understood (or retained) with this version.
-</note>
-<note version="8.3" severity="warning">
-Since Version 8.3, EAGLE supports the association of 3D packages
-with devices in libraries, schematics, and board files. Those 3D
-packages will not be understood (or retained) with this version.
-</note>
 </compatibility>
