File: PCB/PCB/PCB.sch (KiCad schematic (older format))
At the start: 6 parts

Commit message: dsasd
Parts:
- removed J?: Conn_01x02, symbol Connector_Generic:Conn_01x02
- removed U?: NHD-0420H1Z, Display:NHD-0420H1Z, symbol Display_Character:NHD-0420H1Z
- added C1: 10uF, Capacitor_SMD:C_0805_2012Metric, symbol pspice:C
- added C2: 100nF, Capacitor_SMD:C_0805_2012Metric, symbol pspice:C
- added D1, D2, D3, D4, D5, D6: LED, LED_THT:LED_D5.0mm, symbol Device:LED
- added J1: Barrel_Jack_Switch, Connector_BarrelJack:BarrelJack_Horizontal, symbol Connector:Barrel_Jack_Switch
- added J6: SW_ALARM, Connector_PinSocket_2.54mm:PinSocket_1x02_P2.54mm_Vertical, symbol Connector_Generic:Conn_01x02
- added J7: SW_POWER, Connector_PinSocket_2.54mm:PinSocket_1x02_P2.54mm_Vertical, symbol Connector_Generic:Conn_01x02
- added J8: Buzzer, Connector_PinHeader_2.54mm:PinHeader_1x02_P2.54mm_Vertical, symbol Connector_Generic:Conn_01x02
- added Q1: BC548, Package_TO_SOT_THT:TO-92_Inline, symbol Transistor_BJT:BC548
- added R1, R2, R3, R4, R5, R7: 330, Resistor_THT:R_Axial_DIN0918_L18.0mm_D9.0mm_P22.86mm_Horizontal, symbol Device:R
- added R6: 1k, Resistor_THT:R_Axial_DIN0918_L18.0mm_D9.0mm_P22.86mm_Horizontal, symbol pspice:R
- added R8: 1K, Resistor_THT:R_Axial_DIN0918_L18.0mm_D9.0mm_P22.86mm_Horizontal, symbol Device:R
- added RV1, RV3: 10k, Potentiometer_THT:Potentiometer_Bourns_3386F_Vertical, symbol Device:R_POT_TRIM_US
- added RV2: 10k, Potentiometer_THT:Potentiometer_Omeg_PC16BU_Vertical, symbol Device:R_POT_TRIM_US
- added U1: RC1602A, Display:LCD-20x4, symbol Display_Character:RC1602A
- added U2: ULN2803A, Package_DIP:DIP-18_W7.62mm, symbol Transistor_Array:ULN2803A
- added U3: LD1117S33TR_SOT223, Package_TO_SOT_THT:TO-220-3_Vertical, symbol Regulator_Linear:LD1117S33TR_SOT223
- J2, J4: renamed from J?; footprint (none) -> Connector_PinHeader_2.54mm:PinHeader_1x04_P2.54mm_Vertical
- J3: renamed from J?; footprint (none) -> Connector_PinHeader_2.54mm:PinHeader_1x16_P2.54mm_Vertical
- J5: renamed from J?; footprint (none) -> Connector_PinHeader_2.54mm:PinHeader_1x10_P2.54mm_Vertical
Connections:
- net GND: now also J2.2 (Pin_2), J3.13 (Pin_13), J4.2 (Pin_2), C1.2, C2.2, D6.1 (K), J1.1, J8.2 (Pin_2), R6.2, RV1.1, RV2.3, RV3.3, U1.1 (VSS), U1.16 (K), U1.5 (R/W), U2.9 (GND), U3.1 (GND)
- net SDA: now reaches J5.1 (Pin_1)
- net SDA: now also J2.3 (Pin_3), J4.3 (Pin_3)
- net 5V: now reaches J5.10 (Pin_10)
- net 5V: now also J7.1 (Pin_1)
- net SCL: now reaches J5.2 (Pin_2)
- net SCL: now also J2.4 (Pin_4), J4.4 (Pin_4)
- net GPIO14: now reaches J5.3 (Pin_3)
- net GPIO14: now also U1.11 (DB4)
- net GPIO32: now reaches J5.4 (Pin_4)
- net GPIO32: now also U1.12 (DB5)
- net GPIO15: now reaches J5.5 (Pin_5)
- net GPIO15: now also U1.13 (DB6)
- net GPIO33: now reaches J5.6 (Pin_6)
- net GPIO33: now also U1.14 (DB7)
- net GPIO27: now reaches J5.7 (Pin_7)
- net GPIO27: now also U1.6 (E)
- net GPIO12: now reaches J5.8 (Pin_8)
- net GPIO12: now also U1.4 (RS)
- net GPIO13: now reaches J5.9 (Pin_9)
- net GPIO13: now also Q1.2 (B)
- net GPIO21: now reaches J3.1 (Pin_1)
- net GPIO21: now also U2.5 (I5)
- net GPI34: now reaches J3.10 (Pin_10)
- net GPI34: now also J6.2 (Pin_2), R6.1
- net GPIO25: now reaches J3.11 (Pin_11)
- net GPIO25: now also U2.2 (I2)
- net GPIO26: now reaches J3.12 (Pin_12)
- net GPIO26: now also U2.1 (I1)
- net RST: now reaches J3.16 (Pin_16)
- net GPIO17: now reaches J3.2 (Pin_2)
- net GPIO17: now also U2.4 (I4)
- net RX: now reaches J3.3 (Pin_3)
- net GPIO36: now reaches J3.7 (Pin_7)
- net GPIO36: now also U2.3 (I3)
- net GPI35: now reaches J3.8 (Pin_8)
- net GPI35: now also RV2.2
- net GPI39: now reaches J3.9 (Pin_9)
- net 3.3V: now reaches J2.1 (Pin_1)
- net 3.3V: now also J4.1 (Pin_1), C1.1, J6.1 (Pin_1), R1.1, R2.1, R3.1, R4.1, R5.1, R7.1, RV1.3, RV2.1, RV3.1, U1.2 (VDD), U3.2 (VO)
- new net: RV1.2, U1.15 (A/VEE)
- new net: D5.1 (K), U2.14 (O5)
- new net: D4.1 (K), U2.15 (O4)
- new net: D3.1 (K), U2.16 (O3)
- new net: D2.1 (K), U2.17 (O2)
- new net: D1.1 (K), U2.18 (O1)
- new net: D2.2 (A), R2.2
- new net: D3.2 (A), R3.2
- new net: D4.2 (A), R4.2
- new net: D5.2 (A), R5.2
- new net: D1.2 (A), R1.2
- new net: RV3.2, U1.3 (VO)
- new net: Q1.3 (E), R8.2
- new net: D6.2 (A), R7.2
- new net: J8.1 (Pin_1), R8.1
- new net +9V: J1.2, J1.3, Q1.1 (C)
- new net 9V_OUT: C2.1, J7.2 (Pin_2), U3.3 (VI)
- no-connect marks 0 -> 11
